File: schematics/v2/csp_v2.brd (EAGLE design)
At the start: 100 x 67 mm, 61 parts, among them IC1 74AHC1G08DCK, IC2 74HCT04D, IC3 PCA9555PW, IC4 LM339D, J1 2X20-CHIP2X20-SMT-CHIP, U2 DS2431P

Commit message: updated layout
Parts:
- removed BAT1, BAT2, BAT3, BAT4: BTN, wirepad:SMD1,27-2,54
- added G_IN, LR, P_IN, UD: BTN, JKW_CHIP:SMD1,36-3
- moved C12 5.21 mm to (91.7, 12.4), turned to 180 degrees
- moved L- 4.40 mm to (88.2, 10.2)
- moved L+ 3.80 mm to (92.5, 10.2)
Connections:
- net GND: now also G_IN.P$1; no longer BAT4.1
- net N$30: now also UD.P$1; no longer BAT2.1
- net N$31: now also LR.P$1; no longer BAT3.1
- net VCC3V3: now also P_IN.P$1; no longer BAT1.1
Routing:
- net R+OUT: track 101.5 -> 92.7 mm
- net R-OUT: track 105.8 -> 97.2 mm
- net N$38: track 5.01 -> 2.16 mm
- net L-OUT: track 9.46 -> 12.2 mm, vias 0 -> 1
- net GND: track 265.7 -> 263.1 mm, vias 27 -> 28
- net N$31: track 33.2 -> 30.8 mm
- net L+OUT: track 8.31 -> 10.4 mm
- net N$30: track 44.2 -> 42.2 mm
- net VOUT: track 97.9 -> 99.1 mm
- net VCC3V3: track 293.3 -> 293.4 mm, vias 18 -> 20

Commit message: improved v2
Parts:
- moved U$3 3.73 mm to (72.1, 10.5)
- moved C12 3.43 mm to (88.4, 13.5), turned to 90 degrees
- moved C15 1.83 mm to (90.6, 13.5), turned to 270 degrees
- moved U$4 1.66 mm to (61.0, 10.4)
Routing:
- net GND: track 263.1 -> 271.2 mm, vias 28 -> 29
- net AMP_PWR: track 103.3 -> 102.2 mm
